Commit message: implementation: added IMU & altimeter to guppy and worlds

File: install/auv_description/share/auv_description/urdf/cube/camera_module.xacro (robot description, xacro)
@@ -1,58 +1 @@
-<?xml version="1.0"?>
-<robot name="camera_module" xmlns:xacro="http://ros.org/wiki/xacro">
-  <!-- Camera with optical frame + Gazebo SDF sensor -->
-  <xacro:macro name="camera_module"
-               params="parent link_name optical_frame
-                       box
-                       mount_xyz mount_rpy
-                       horiz_fov img_w img_h topic update_rate visualize">
-    <!-- Parse box vector -->
-    <xacro:property name="bx" value="${box.split()[0]}"/>
-    <xacro:property name="by" value="${box.split()[1]}"/>
-    <xacro:property name="bz" value="${box.split()[2]}"/>
-    <link name="${link_name}">
-      <visual>
-        <geometry><box size="${bx} ${by} ${bz}"/></geometry>
-        <material name="black"><color rgba="0 0 0 1"/></material>
-      </visual>
-      <collision>
-        <geometry><box size="${bx} ${by} ${bz}"/></geometry>
-      </collision>
-      <inertial>
-        <mass value="0.1"/>
-        <inertia ixx="8.333e-4" iyy="8.333e-4" izz="8.333e-4" ixy="0" ixz="0" iyz="0"/>
-      </inertial>
-    </link>
-    <joint name="${link_name}_mount" type="fixed">
-      <parent link="${parent}"/>
-      <child link="${link_name}"/>
-      <origin xyz="${mount_xyz}" rpy="${mount_rpy}"/>
-    </joint>
-    <!-- REP-103 optical frame (z forward, x right, y down) -->
-    <link name="${optical_frame}"/>
-    <joint name="${optical_frame}_joint" type="fixed">
-      <parent link="${link_name}"/>
-      <child link="${optical_frame}"/>
-      <origin xyz="0 0 0" rpy="-1.57079632679 0 -1.57079632679"/>
-    </joint>
-    <!-- Gazebo sensor on camera_link -->
-    <gazebo reference="${link_name}">
-      <sensor name="${link_name}_sensor" type="camera">
-        <pose>0 0 0 0 0 0</pose>
-        <always_on>true</always_on>
-        <update_rate>${update_rate}</update_rate>
-        <visualize>${visualize}</visualize>
-        <camera>
-          <horizontal_fov>${horiz_fov}</horizontal_fov>
-          <image>
-            <width>${img_w}</width>
-            <height>${img_h}</height>
-            <format>R8G8B8</format>
-          </image>
-          <clip><near>0.1</near><far>100</far></clip>
-        </camera>
-        <topic>${topic}</topic>
-      </sensor>
-    </gazebo>
-  </xacro:macro>
-</robot>
+/home/sangregorioquimpo/auve2_ws/src/auv_description/urdf/cube/camera_module.xacro

File: install/auv_description/share/auv_description/urdf/cube/cube_link.xacro (robot description, xacro)
@@ -1,22 +1 @@
-<?xml version="1.0"?>
-<robot name="cube_module" xmlns:xacro="http://ros.org/wiki/xacro">
-  <!-- Box inertia helper (I = 1/12 m (y^2+z^2), etc.) -->
-  <xacro:macro name="cube_base" params="name size_x size_y size_z mass">
-    <xacro:property name="ixx" value="${(1.0/12.0) * mass * (pow(size_y,2) + pow(size_z,2))}"/>
-    <xacro:property name="iyy" value="${(1.0/12.0) * mass * (pow(size_x,2) + pow(size_z,2))}"/>
-    <xacro:property name="izz" value="${(1.0/12.0) * mass * (pow(size_x,2) + pow(size_y,2))}"/>
-    <link name="${name}">
-      <visual>
-        <geometry><box size="${size_x} ${size_y} ${size_z}"/></geometry>
-        <material name="blue"><color rgba="0 0 1 1"/></material>
-      </visual>
-      <collision>
-        <geometry><box size="${size_x} ${size_y} ${size_z}"/></geometry>
-      </collision>
-      <inertial>
-        <mass value="${mass}"/>
-        <inertia ixx="${ixx}" iyy="${iyy}" izz="${izz}" ixy="0" ixz="0" iyz="0"/>
-      </inertial>
-    </link>
-  </xacro:macro>
-</robot>
+/home/sangregorioquimpo/auve2_ws/src/auv_description/urdf/cube/cube_link.xacro

File: install/auv_description/share/auv_description/urdf/cube/lidar3d_module.xacro (robot description, xacro)
@@ -1,65 +1 @@
-<?xml version="1.0"?>
-<robot name="lidar3d_module" xmlns:xacro="http://ros.org/wiki/xacro">
-  <!-- 3D LiDAR (gpu_lidar) producing a point cloud.
-       Defaults match the tutorial's 3D lidar (VLP-32-like) vertical span.
-       Bridge with:
-         /scan/points@sensor_msgs/msg/PointCloud2@gz.msgs.PointCloudPacked
-  -->
-  <xacro:macro name="lidar3d_module"
-               params="parent link_name
-                       mount_xyz:='0.55 0 0.2' mount_rpy:='0 0 0'
-                       radius:='0.05' length:='0.10' mass:='0.25'
-                       topic:='/lidar/points' update_rate:='10'
-                       range_min:='0.2' range_max:='50.0'
-                       h_samples:='1024' h_min:='-3.14159' h_max:='3.14159'
-                       v_samples:='32'   v_min:='-0.5353'  v_max:='0.1862'">
-    <!-- Body -->
-    <link name="${link_name}">
-      <visual>
-        <geometry><cylinder radius="${radius}" length="${length}"/></geometry>
-        <material name="darkgray"><color rgba="0.3 0.3 0.3 1"/></material>
-      </visual>
-      <collision>
-        <geometry><cylinder radius="${radius}" length="${length}"/></geometry>
-      </collision>
-      <inertial>
-        <mass value="${mass}"/>
-        <inertia ixx="0.001" iyy="0.001" izz="0.001" ixy="0" ixz="0" iyz="0"/>
-      </inertial>
-    </link>
-    <joint name="${link_name}_mount" type="fixed">
-      <parent link="${parent}"/>
-      <child  link="${link_name}"/>
-      <origin xyz="${mount_xyz}" rpy="${mount_rpy}"/>
-    </joint>
-    <!-- Gazebo Harmonic 3D LiDAR -->
-    <gazebo reference="${link_name}">
-      <sensor name="${link_name}_sensor" type="gpu_lidar">
-        <always_on>true</always_on>
-        <update_rate>${update_rate}</update_rate>
-        <visualize>true</visualize>
-        <lidar>
-          <scan>
-            <horizontal>
-              <samples>${h_samples}</samples>
-              <min_angle>${h_min}</min_angle>
-              <max_angle>${h_max}</max_angle>
-            </horizontal>
-            <vertical>
-              <samples>${v_samples}</samples>
-              <min_angle>${v_min}</min_angle>
-              <max_angle>${v_max}</max_angle>
-            </vertical>
-          </scan>
-          <range>
-            <min>${range_min}</min>
-            <max>${range_max}</max>
-            <resolution>0.01</resolution>
-          </range>
-        </lidar>
-        <!-- Gazebo Transport point cloud topic (per tutorial: /scan/points) -->
-        <topic>${topic}</topic>
-      </sensor>
-    </gazebo>
-  </xacro:macro>
-</robot>
+/home/sangregorioquimpo/auve2_ws/src/auv_description/urdf/cube/lidar3d_module.xacro

File: install/auv_description/share/auv_description/urdf/cube/plugins.xacro (robot description, xacro)
@@ -1,26 +1 @@
-<?xml version="1.0"?>
-<robot name="plugins_module" xmlns:xacro="http://ros.org/wiki/xacro">
-  <xacro:macro name="buoyancy_plugin" params="link_name water_level fluid_density volume">
-    <gazebo>
-      <plugin filename="libsimple_buoyancy.so" name="gz::sim::systems::SimpleBuoyancy">
-        <link_name>${link_name}</link_name>
-        <water_level>${water_level}</water_level>
-        <fluid_density>${fluid_density}</fluid_density>
-        <volume>${volume}</volume>
-      </plugin>
-    </gazebo>
-  </xacro:macro>
-  <xacro:macro name="wasd_plugin" params="link_name topic">
-    <gazebo>
-      <plugin name="wasd_body_thrust_plugin" filename="libwasd_body_thrust_plugin.so">
-        <link_name>${link_name}</link_name>
-        <topic>${topic}</topic>
-        <lever>0 0 0</lever>
-        <hold_ms>-1</hold_ms>
-        <scale>1.0</scale>
-        <force_scale>1.0</force_scale>
-        <torque_scale>1.0</torque_scale>
-      </plugin>
-    </gazebo>
-  </xacro:macro>
-</robot>
+/home/sangregorioquimpo/auve2_ws/src/auv_description/urdf/cube/plugins.xacro

File: install/auv_description/share/auv_description/urdf/guppy/plugins.xacro (robot description, xacro)
@@ -1,25 +1 @@
-<?xml version="1.0"?>
-<robot name="plugins_module" xmlns:xacro="http://ros.org/wiki/xacro">
-  <xacro:macro name="buoyancy_plugin" params="link_name water_level fluid_density volume">
-    <gazebo>
-      <plugin filename="libsimple_buoyancy.so" name="gz::sim::systems::SimpleBuoyancy">
-        <link_name>${link_name}</link_name>
-        <water_level>${water_level}</water_level>
-        <fluid_density>${fluid_density}</fluid_density>
-        <volume>${volume}</volume>
-      </plugin>
-    </gazebo>
-  </xacro:macro>
-  <xacro:macro name="wasd_plugin" params="link_name topic">
-    <gazebo>
-      <plugin name="wasd_body_thrust_plugin" filename="libwasd_body_thrust_plugin.so">
-        <link_name>${link_name}</link_name>
-        <topic>${topic}</topic>
-        <hold_ms>-1</hold_ms>
-        <scale>1.0</scale>
-        <force_scale>1.0</force_scale>
-        <torque_scale>1.0</torque_scale>
-      </plugin>
-    </gazebo>
-  </xacro:macro>
-</robot>
+/home/sangregorioquimpo/auve2_ws/src/auv_description/urdf/guppy/plugins.xacro

File: src/auv_description/urdf/guppyExperimental/guppytest1Experimental.urdf (robot description, URDF)
Before this commit: robot guppytest1, 9 links, 8 joints
Links:
- added link imu_link, mass 0.01; collision box size=0.01 0.01 0.01; visual box size=0.01 0.01 0.01
Joints:
- added joint imu_joint: type fixed, parent base_link, child imu_link, origin xyz=0 0 0.05 rpy=0 0 0
